Commit message: update the new enviornment

File: examples/compass_gait/cart.urdf (robot description, URDF)
Before this commit: robot locobot, 25 links, 24 joints
Joints:
- joint base_joint: origin xyz=2 6.5 2 rpy=0 0 -0.5 -> xyz=-9 0 -0.7 rpy=0 0 -0.5

File: examples/compass_gait/cart1.urdf (robot description, URDF)
Before this commit: robot locobot, 25 links, 24 joints
Joints:
- joint base_joint: origin xyz=0 2.5 2 rpy=0 0 0 -> xyz=-3 -3.5 -0.7 rpy=0 0 1.57

File: examples/compass_gait/cart2.urdf (robot description, URDF)
Before this commit: robot locobot, 25 links, 24 joints
Joints:
- joint base_joint: origin xyz=3 -3 1 rpy=0 0 0.5 -> xyz=-6 -9 -1.7 rpy=0 0 0.5
