Commit message: running

File: examples/KneedCompassGait/KneedCompassGait.urdf (robot description, URDF)
Before this commit: robot KneedCompassGait, 9 links, 8 joints
Links:
- link left_lower_leg: geometry collision sphere radius=0; collision sphere radius=0
- link right_lower_leg: geometry collision sphere radius=0; collision sphere radius=0
Joints:
- joint left_knee_pin: limit lower=0 effort=100 -> lower=-3.14 upper=0
- joint right_knee_pin: limit lower=0 effort=100 -> lower=-3.14 upper=0

Commit message: Finished QP controller

File: examples/KneedCompassGait/KneedCompassGait.urdf (robot description, URDF)
Before this commit: robot KneedCompassGait, 9 links, 8 joints
Joints:
- joint hip_pin: limit (none) -> effort=200
- joint left_knee_pin: limit lower=-3.14 upper=0 -> lower=-3.14 upper=0 effort=100
- joint right_knee_pin: limit lower=-3.14 upper=0 -> lower=-3.14 upper=0 effort=100

Commit message: update kneed compass gait and construct the cassie scenario

File: examples/KneedCompassGait/KneedCompassGait.urdf (robot description, URDF)
Before this commit: robot KneedCompassGait, 9 links, 8 joints
Links:
- added link base_link
- added link hip2pin
- added link pin2yaw
- link left_lower_leg: geometry collision sphere radius=0; visual cylinder length=0.5 radius=0.0075
- link right_lower_leg: geometry collision sphere radius=0; visual cylinder length=0.5 radius=0.0075
Joints:
- added joint base: type fixed, parent base_link, child hip
- added joint hip_roll: type continuous, parent hip, child hip2pin, axis 1 0 0, limit effort=200 velocity=100
- added joint hip_yaw: type continuous, parent pin2yaw, child right_upper_leg, axis 0 0 1, limit effort=200 velocity=100
- joint hip_pin: child right_upper_leg -> pin2yaw; limit effort=200 -> effort=200 velocity=100; parent hip -> hip2pin
- joint left_knee_pin: limit lower=-3.14 upper=0 effort=100 -> lower=-3.14 upper=0 effort=100 velocity=100
- joint right_knee_pin: limit lower=-3.14 upper=0 effort=100 -> lower=-3.14 upper=0 effort=100 velocity=100

Commit message: one step trail

File: examples/KneedCompassGait/KneedCompassGait.urdf (robot description, URDF)
Before this commit: robot KneedCompassGait, 12 links, 11 joints
Joints:
- joint left_knee_pin: limit lower=-3.14 upper=0 effort=100 velocity=100 -> lower=-3.14 upper=0 effort=200 velocity=100
- joint right_knee_pin: limit lower=-3.14 upper=0 effort=100 velocity=100 -> lower=-3.14 upper=0 effort=200 velocity=100

Commit message: MPC like manually QP

File: examples/KneedCompassGait/KneedCompassGait.urdf (robot description, URDF)
Before this commit: robot KneedCompassGait, 12 links, 11 joints
Joints:
- joint hip_pin: limit effort=200 velocity=100 -> effort=1000 velocity=100
- joint left_knee_pin: limit lower=-3.14 upper=0 effort=200 velocity=100 -> lower=-3.14 upper=0 effort=1000 velocity=100
- joint right_knee_pin: limit lower=-3.14 upper=0 effort=200 velocity=100 -> lower=-3.14 upper=0 effort=1000 velocity=100

Commit message: added a line-hip and trying to control it

File: examples/KneedCompassGait/KneedCompassGait.urdf (robot description, URDF)
Before this commit: robot KneedCompassGait, 12 links, 11 joints
Links:
- removed link hip
- removed link hip2pin
- removed link pin2yaw
- added link hip_line; visual cylinder length=0.2 radius=0.0075
- added link hip_mass, mass 10; visual sphere radius=0.05
- added link right_hip2roll
Joints:
- removed joint hip_pin
- removed joint hip_roll
- removed joint hip_yaw
- removed joint left_leg_weld
- added joint hip_mass_weld: type fixed, parent hip_line, child hip_mass
- added joint leftHip_roll: type continuous, parent hip_line, child left_upper_leg, origin xyz=0 0 0.1 rpy=-1.5708 0 0, axis 1 0 0, limit effort=200 velocity=100
- added joint rightHip_pin: type continuous, parent right_hip2roll, child right_upper_leg, axis 0 1 0, limit effort=200 velocity=100
- added joint rightHip_roll: type continuous, parent hip_line, child right_hip2roll, origin xyz=0 0 -0.1 rpy=-1.5708 0 0, axis 1 0 0, limit effort=200 velocity=100
- joint base: child hip -> hip_line; origin (none) -> xyz=0 0 0 rpy=1.5708 0 0

Commit message: line inertial hip, yaw control

File: examples/KneedCompassGait/KneedCompassGait.urdf (robot description, URDF)
Before this commit: robot KneedCompassGait, 12 links, 11 joints
Links:
- removed link hip_mass
- added link left_hip2roll
- link hip_line: mass None -> 10
Joints:
- removed joint hip_mass_weld
- added joint leftHip_pin: type continuous, parent left_hip2roll, child left_upper_leg, axis 0 1 0, limit effort=200 velocity=100
- joint leftHip_roll: child left_upper_leg -> left_hip2roll

Commit message: commented version

File: examples/KneedCompassGait/KneedCompassGait.urdf (robot description, URDF)
Before this commit: robot KneedCompassGait, 12 links, 11 joints
Links:
- link hip_line: geometry visual cylinder length=0.2 radius=0.003; visual cylinder length=0.2 radius=0.0075
